Commit message: piper: define TCP at gripper contact point (piper_tcp), not the wrist
The agent used ee_link_name="link6" (the wrist flange) as the TCP, but the
gripper fingers extend ~0.136m forward of link6. The PushCube/PickCube dense
reward drives the TCP to behind/beside the cube, so with the wrist as TCP the
gripper ended up ~0.13m PAST the cube (goal side) and jammed -- the arm could
never push/grasp (success stayed 0).

Fix: add a massless piper_tcp link fixed to gripper_base at xyz="0 0 0.1358"
(the fingertip/contact line, analogous to panda_hand_tcp) and point
ee_link_name at it. Verified on CPU: piper_tcp registers, TCP now sits at the
gripper front (0.133m forward of the wrist), the push target behind the cube
is reachable, env loads/steps cleanly.

Co-Authored-By: Claude <noreply@anthropic.com>

File: mani_skill/assets/robots/piper/piper_description.urdf (robot description, URDF)
Before this commit: robot piper, 10 links, 9 joints
Links:
- added link piper_tcp
Joints:
- added joint piper_tcp_joint: type fixed, parent gripper_base, child piper_tcp, origin xyz=0 0 0.1358 rpy=0 0 0
